Commit message: Implement four-wheeled robot model with sensors and control logic; add launch files and world configuration for simulation

File: urdf/robot.xacro (robot description, xacro)
@@ -61,14 +61,32 @@
     <link name="${name}">
       <visual>
-        <!-- TODO: Complete -->
+        <geometry>
+          <cylinder radius="${wheel_link_radius}" length="${wheel_link_length}"/>
+        </geometry>
+        <origin rpy="1.5708 0 0" xyz="0 0 0"/>
+        <material name="wheel_material">
+          <color rgba="0.2 0.2 0.2 1"/>
+        </material>
       </visual>
       <collision>
-        <!-- TODO: Complete -->
+        <geometry>
+          <cylinder radius="${wheel_link_radius}" length="${wheel_link_length}"/>
+        </geometry>
+        <origin rpy="1.5708 0 0" xyz="0 0 0"/>
       </collision>
       <inertial>
-        <!-- TODO: Complete -->
+        <origin rpy="1.5708 0 0" xyz="0 0 0"/>
+        <mass value="${wheel_mass}"/>
+        <inertia
+          ixx="${I_wheel}" ixy="0" ixz="0"
+          iyy="${I_wheel}" iyz="0"
+          izz="${Iz_wheel}"/>
+      </inertial>
     </link>
     <joint name="${name}_joint" type="${joint_type}">
-      <!-- TODO: Complete -->
+      <parent link="body_link"/>
+      <child link="${name}"/>
+      <origin xyz="${x} ${y} ${z}"/>
+      <axis xyz="0 1 0"/>
       <limit effort="1000" velocity="1000"/>
       <dynamics damping="1.0" friction="1.0"/>
@@ -77,10 +95,15 @@
   <!-- Instantiate wheels -->
   <xacro:wheel name="rear_right_wheel"  x="${-body_link_x_dim/2 + 1.2*wheel_link_radius}" y="${-body_link_y_dim/2 - 1.2*wheel_link_length/2}" z="${wheel_link_z_location}" joint_type="continuous"/>
-  <!-- TODO: Complete: Wheels must be named - rear_left_wheel, front_right_wheel, front_left_wheel -->
-<!-- Camera -->
+  <xacro:wheel name="rear_left_wheel"   x="${-body_link_x_dim/2 + 1.2*wheel_link_radius}" y="${body_link_y_dim/2 + 1.2*wheel_link_length/2}" z="${wheel_link_z_location}" joint_type="continuous"/>
+  <xacro:wheel name="front_right_wheel" x="${body_link_x_dim/2 - 1.2*wheel_link_radius}" y="${-body_link_y_dim/2 - 1.2*wheel_link_length/2}" z="${wheel_link_z_location}" joint_type="continuous"/>
+  <xacro:wheel name="front_left_wheel"  x="${body_link_x_dim/2 - 1.2*wheel_link_radius}" y="${body_link_y_dim/2 + 1.2*wheel_link_length/2}" z="${wheel_link_z_location}" joint_type="continuous"/>
+  <!-- Camera -->
   <link name="camera_link">
     <visual>
       <geometry><box size="${sensor_side} ${sensor_side} ${sensor_side}"/></geometry>
       <origin rpy="0 0 0" xyz="0 0 0" />
+      <material name="camera_material">
+        <color rgba="0.0 0.0 1.0 1"/>
+      </material>
     </visual>
     <collision>
@@ -100,20 +123,62 @@
     <parent link="body_link"/>
     <child link="camera_link"/>
-    <origin xyz="${-body_link_x_dim/4} 0 ${body_link_z_dim/2 + sensor_side/2}"/>
+    <origin xyz="${body_link_x_dim/2} 0 ${body_link_z_dim/2 + sensor_side/2}"/>
     <axis xyz="0 1 0" />
   </joint>
   <!-- Sonar -->
   <link name="sonar_link">
-    <!-- TODO: Complete -->
+    <visual>
+      <geometry><box size="${sensor_side} ${sensor_side} ${sensor_side}"/></geometry>
+      <origin rpy="0 0 0" xyz="0 0 0" />
+      <material name="sonar_material">
+        <color rgba="1.0 0.0 0.0 1"/>
+      </material>
+    </visual>
+    <collision>
+      <geometry><box size="${sensor_side} ${sensor_side} ${sensor_side}"/></geometry>
+      <origin rpy="0 0 0" xyz="0 0 0" />
+    </collision>
+    <inertial>
+      <origin rpy="0 0 0" xyz="0 0 0"/>
+      <mass value="${sensor_mass}"/>
+      <inertia
+        ixx="1e-6" ixy="0.0" ixz="0.0"
+        iyy="1e-6" iyz="0.0"
+        izz="1e-6"/>
+    </inertial>
   </link>
   <joint name="sonar_joint" type="fixed">
-    <!-- TODO: Complete -->
+    <parent link="body_link"/>
+    <child link="sonar_link"/>
+    <origin xyz="${body_link_x_dim/2} ${body_link_y_dim/4} ${body_link_z_dim/2 + sensor_side/2}"/>
+    <axis xyz="0 1 0" />
   </joint>
   <!-- Lidar -->
   <link name="lidar_link">
-    <!-- TODO: Complete -->
+    <visual>
+      <geometry><cylinder radius="${sensor_side}" length="${sensor_side}"/></geometry>
+      <origin rpy="0 0 0" xyz="0 0 0" />
+      <material name="lidar_material">
+        <color rgba="0.0 1.0 0.0 1"/>
+      </material>
+    </visual>
+    <collision>
+      <geometry><cylinder radius="${sensor_side}" length="${sensor_side}"/></geometry>
+      <origin rpy="0 0 0" xyz="0 0 0" />
+    </collision>
+    <inertial>
+      <origin rpy="0 0 0" xyz="0 0 0"/>
+      <mass value="${sensor_mass}"/>
+      <inertia
+        ixx="1e-6" ixy="0.0" ixz="0.0"
+        iyy="1e-6" iyz="0.0"
+        izz="1e-6"/>
+    </inertial>
   </link>
   <joint name="lidar_joint" type="fixed">
-    <!-- TODO: Complete -->
+    <parent link="body_link"/>
+    <child link="lidar_link"/>
+    <origin xyz="0 0 ${body_link_z_dim/2 + sensor_side/2}"/>
+    <axis xyz="0 1 0" />
   </joint>
 </robot>
